File: ESP8266/Eagle/AtmoOrb/AtmoOrb.sch (EAGLE design)
At the start: 10 parts, among them J1 DCJ0202

Commit message: Added a switch to bring ESP8266 into update mode to schematic and board layout
Parts:
- added S1: TL32PO, switch:TL32PO
Connections:
- new net N$6: ESP8266.GPIO0, S1.P
- net GND: now also S1.S
Changed lines of the file:
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@@
 <part name="+3V2" library="supply1" deviceset="+3V3" device=""/>
 <part name="ESP8266" library="ESP8266" deviceset="ESP8266" device=""/>
+<part name="S1" library="switch" deviceset="TL32PO" device=""/>
 </parts>
 <sheets>
@@
 <instance part="+3V2" gate="G$1" x="111.76" y="104.14"/>
 <instance part="ESP8266" gate="G$1" x="132.08" y="91.44"/>
+<instance part="S1" gate="BEF1" x="170.18" y="88.9" rot="R270"/>
 </instances>
 <busses>
@@
 <segment>
 <wire x1="149.86" y1="93.98" x2="157.48" y2="93.98" width="0.1524" layer="91"/>
-<wire x1="157.48" y1="93.98" x2="157.48" y2="81.28" width="0.1524" layer="91"/>
+<wire x1="157.48" y1="93.98" x2="157.48" y2="83.82" width="0.1524" layer="91"/>
 <pinref part="GND8" gate="1" pin="GND"/>
 <pinref part="ESP8266" gate="G$1" pin="GND"/>
+<wire x1="157.48" y1="83.82" x2="157.48" y2="81.28" width="0.1524" layer="91"/>
+<wire x1="175.26" y1="86.36" x2="177.8" y2="86.36" width="0.1524" layer="91"/>
+<wire x1="177.8" y1="86.36" x2="177.8" y2="83.82" width="0.1524" layer="91"/>
+<wire x1="177.8" y1="83.82" x2="157.48" y2="83.82" width="0.1524" layer="91"/>
+<junction x="157.48" y="83.82"/>
+<pinref part="S1" gate="BEF1" pin="S"/>
 </segment>
 </net>
@@
 </segment>
 </net>
+<net name="N$6" class="0">
+<segment>
+<pinref part="ESP8266" gate="G$1" pin="GPIO0"/>
+<wire x1="149.86" y1="88.9" x2="165.1" y2="88.9" width="0.1524" layer="91"/>
+<pinref part="S1" gate="BEF1" pin="P"/>
+</segment>
+</net>
